File: 8080-HC.kicad_pcb (KiCad board)
At the start: 4 copper layers, 354 parts, among them U1 74HCU04, U10 74HC00, U11 74HC126, U12 74HC161, U13 74HC238, U14 74HC238, U15 74HC238, U16 74HC238, U17 74HC04, U178 74LS03, U18 74HC05, U180 74HC244, U181 74HC244, U182 74HC244, U19 74HC74, U193 74HC244, U194 74HC244, U195 74HC244, U2 74HC74, U20 74HC373, U21 74HC373, U214 74HC373, U215 74HC193, U216 74HC193, U217 74HC193, U218 74HC193, U22 74HC373, U227 74HC04, U228 74HC04, U229 74HC04, U23 74HC373, U230 74HC04, U231 74HC245, U232 74HC04, U233 74HC04, U234 74LS373, U239 74HC74, U24 74HC373, U242 74HC00, U243 74HCU04, U244 74HC00, U25 74HC244, U26 74HC244, U27 74HC244, U28 74HC244, U29 74HC244, U3 74HC00, U30 74HC373, U31 74HC373, U32 74HC244, U33 74HC244, U34 74HC244, U35 74HC244, U36 74HC373, U38 74HC244, U39 74HC244, U4 74HC04, U48 74HC04, U49 74HC04, U5 74HC00, U50 74HC04, U51 74HC04, U52 74HC04, U53 74HC238, U54 74HC238, U55 74HC238, U56 74HC238, U57 74HC04, U58 74HC04, U6 74HC04, U69 74HC05, U7 74HC05, U70 74LS05, U71 74HC04, U72 74LS126, U73 74LS126, U74 74LS126, U75 74LS126, U76 74LS126, U77 74HC00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

Commit message: move a couple of components to cleanup ratsnets
Parts:
- moved B5 303.9 mm to (-424.1, -18.7), turned to 90 degrees
- moved B41 266.2 mm to (-420.9, -18.8)
- moved B43 18.6 mm to (-428.3, -12.0)
Changed lines of the file:
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@@
   )
   (module Resistor_THT:R_Array_SIP9 (layer F.Cu)
-    (at -361.95 -316.23)
-    (descr "9-pin Resistor SIP pack")
-    (tags R)
-    (fp_text reference B5 (at 11.43 -2.4) (layer F.SilkS)
-      (effects (font (size 1 1) (thickness 0.15)))
-    )
-    (fp_text value 1K (at 11.43 2.4) (layer F.Fab)
-      (effects (font (size 1 1) (thickness 0.15)))
-    )
-    (fp_line (start 22.05 -1.65) (end -1.7 -1.65) (layer F.CrtYd) (width 0.05))
-    (fp_line (start 22.05 1.65) (end 22.05 -1.65) (layer F.CrtYd) (width 0.05))
-    (fp_line (start -1.7 1.65) (end 22.05 1.65) (layer F.CrtYd) (width 0.05))
-    (fp_line (start -1.7 -1.65) (end -1.7 1.65) (layer F.CrtYd) (width 0.05))
-    (fp_line (start 1.27 -1.4) (end 1.27 1.4) (layer F.SilkS) (width 0.12))
-    (fp_line (start 21.76 -1.4) (end -1.44 -1.4) (layer F.SilkS) (width 0.12))
-    (fp_line (start 21.76 1.4) (end 21.76 -1.4) (layer F.SilkS) (width 0.12))
-    (fp_line (start -1.44 1.4) (end 21.76 1.4) (layer F.SilkS) (width 0.12))
-    (fp_line (start -1.44 -1.4) (end -1.44 1.4) (layer F.SilkS) (width 0.12))
-    (fp_line (start 1.27 -1.25) (end 1.27 1.25) (layer F.Fab) (width 0.1))
-    (fp_line (start 21.61 -1.25) (end -1.29 -1.25) (layer F.Fab) (width 0.1))
-    (fp_line (start 21.61 1.25) (end 21.61 -1.25) (layer F.Fab) (width 0.1))
-    (fp_line (start -1.29 1.25) (end 21.61 1.25) (layer F.Fab) (width 0.1))
-    (fp_line (start -1.29 -1.25) (end -1.29 1.25) (layer F.Fab) (width 0.1))
-    (fp_text user %R (at 10.16 0) (layer F.Fab)
-      (effects (font (size 1 1) (thickness 0.15)))
-    )
-    (pad 9 thru_hole oval (at 20.32 0) (size 1.6 1.6) (drill 0.8) (layers *.Cu *.Mask)
+    (at -424.1165 -18.7325 90)
+    (descr "9-pin Resistor SIP pack")
+    (tags R)
+    (fp_text reference B5 (at 11.43 -2.4 90) (layer F.SilkS)
+      (effects (font (size 1 1) (thickness 0.15)))
+    )
+    (fp_text value 1K (at 11.43 2.4 90) (layer F.Fab)
+      (effects (font (size 1 1) (thickness 0.15)))
+    )
+    (fp_line (start 22.05 -1.65) (end -1.7 -1.65) (layer F.CrtYd) (width 0.05))
+    (fp_line (start 22.05 1.65) (end 22.05 -1.65) (layer F.CrtYd) (width 0.05))
+    (fp_line (start -1.7 1.65) (end 22.05 1.65) (layer F.CrtYd) (width 0.05))
+    (fp_line (start -1.7 -1.65) (end -1.7 1.65) (layer F.CrtYd) (width 0.05))
+    (fp_line (start 1.27 -1.4) (end 1.27 1.4) (layer F.SilkS) (width 0.12))
+    (fp_line (start 21.76 -1.4) (end -1.44 -1.4) (layer F.SilkS) (width 0.12))
+    (fp_line (start 21.76 1.4) (end 21.76 -1.4) (layer F.SilkS) (width 0.12))
+    (fp_line (start -1.44 1.4) (end 21.76 1.4) (layer F.SilkS) (width 0.12))
+    (fp_line (start -1.44 -1.4) (end -1.44 1.4) (layer F.SilkS) (width 0.12))
+    (fp_line (start 1.27 -1.25) (end 1.27 1.25) (layer F.Fab) (width 0.1))
+    (fp_line (start 21.61 -1.25) (end -1.29 -1.25) (layer F.Fab) (width 0.1))
+    (fp_line (start 21.61 1.25) (end 21.61 -1.25) (layer F.Fab) (width 0.1))
+    (fp_line (start -1.29 1.25) (end 21.61 1.25) (layer F.Fab) (width 0.1))
+    (fp_line (start -1.29 -1.25) (end -1.29 1.25) (layer F.Fab) (width 0.1))
+    (fp_text user %R (at 10.16 0 90) (layer F.Fab)
+      (effects (font (size 1 1) (thickness 0.15)))
+    )
+    (pad 9 thru_hole oval (at 20.32 0 90) (size 1.6 1.6) (drill 0.8) (layers *.Cu *.Mask)
       (net 354 iB7))
-    (pad 8 thru_hole oval (at 17.78 0) (size 1.6 1.6) (drill 0.8) (layers *.Cu *.Mask)
+    (pad 8 thru_hole oval (at 17.78 0 90) (size 1.6 1.6) (drill 0.8) (layers *.Cu *.Mask)
       (net 356 iB6))
-    (pad 7 thru_hole oval (at 15.24 0) (size 1.6 1.6) (drill 0.8) (layers *.Cu *.Mask)
+    (pad 7 thru_hole oval (at 15.24 0 90) (size 1.6 1.6) (drill 0.8) (layers *.Cu *.Mask)
       (net 358 iB5))
-    (pad 6 thru_hole oval (at 12.7 0) (size 1.6 1.6) (drill 0.8) (layers *.Cu *.Mask)
+    (pad 6 thru_hole oval (at 12.7 0 90) (size 1.6 1.6) (drill 0.8) (layers *.Cu *.Mask)
       (net 360 iB4))
-    (pad 5 thru_hole oval (at 10.16 0) (size 1.6 1.6) (drill 0.8) (layers *.Cu *.Mask)
+    (pad 5 thru_hole oval (at 10.16 0 90) (size 1.6 1.6) (drill 0.8) (layers *.Cu *.Mask)
       (net 361 iB3))
-    (pad 4 thru_hole oval (at 7.62 0) (size 1.6 1.6) (drill 0.8) (layers *.Cu *.Mask)
+    (pad 4 thru_hole oval (at 7.62 0 90) (size 1.6 1.6) (drill 0.8) (layers *.Cu *.Mask)
       (net 359 iB2))
-    (pad 3 thru_hole oval (at 5.08 0) (size 1.6 1.6) (drill 0.8) (layers *.Cu *.Mask)
+    (pad 3 thru_hole oval (at 5.08 0 90) (size 1.6 1.6) (drill 0.8) (layers *.Cu *.Mask)
       (net 357 iB1))
-    (pad 2 thru_hole oval (at 2.54 0) (size 1.6 1.6) (drill 0.8) (layers *.Cu *.Mask)
+    (pad 2 thru_hole oval (at 2.54 0 90) (size 1.6 1.6) (drill 0.8) (layers *.Cu *.Mask)
       (net 355 iB0))
-    (pad 1 thru_hole rect (at 0 0) (size 1.6 1.6) (drill 0.8) (layers *.Cu *.Mask)
+    (pad 1 thru_hole rect (at 0 0 90) (size 1.6 1.6) (drill 0.8) (layers *.Cu *.Mask)
       (net 3 VCC))
     (model ${KISYS3DMOD}/Resistor_THT.3dshapes/R_Array_SIP9.wrl
@@
   )
   (module Resistor_THT:R_Array_SIP9 (layer F.Cu)
-    (at -436.88 -284.48 90)
+    (at -420.878 -18.796 90)
     (descr "9-pin Resistor SIP pack")
     (tags R)
@@
   )
   (module Resistor_THT:R_Array_SIP9 (layer F.Cu)
-    (at -424.688 -30.226 270)
-    (descr "9-pin Resistor SIP pack")
-    (tags R)
+    (at -428.3075 -12.0015 270)
+    (descr "9-pin Resistor SIP pack")
+    (tags R)
