File: HALT.sch (KiCad schematic (older format))
At the start: 8 parts, among them U244 74HC00, U3 74HC00, U49 74HC04, U84 74HC03, U88 74HC126, U91 74HC00

Commit message: route A8-A15 to U131
Parts:
- R44: footprint Resistor_THT:R_Axial_DIN0207_L6.3mm_D2.5mm_P10.16mm_Horizontal -> Resistor_THT:R_Axial_DIN0204_L3.6mm_D1.6mm_P5.08mm_Horizontal
Changed lines of the file:
@@
 F 0 "R44" H 6170 1496 50  0000 L CNN
 F 1 "R" H 6170 1405 50  0000 L CNN
-F 2 "Resistor_THT:R_Axial_DIN0207_L6.3mm_D2.5mm_P10.16mm_Horizontal" V 6030 1450 50  0001 C CNN
+F 2 "Resistor_THT:R_Axial_DIN0204_L3.6mm_D1.6mm_P5.08mm_Horizontal" V 6030 1450 50  0001 C CNN
 F 3 "~" H 6100 1450 50  0001 C CNN
 	1    6100 1450
