File: IO_control_signals.sch (KiCad schematic (older format))
At the start: 32 parts, among them U242 74HC00, U244 74HC00, U3 74HC00, U58 74HC04, U69 74HC05, U70 74LS05, U71 74HC04, U72 74LS126, U73 74LS126, U74 74LS126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

Commit message: route the iBn bus on the left side of the board
Parts:
- renumbered R37 to R937, R38 to R938
Changed lines of the file:
@@
 ioWR
 $Comp
-L Device:R R37
+L Device:R R937
 U 1 1 610ACAB0
 P 4750 2800
-F 0 "R37" H 4820 2846 50  0000 L CNN
+F 0 "R937" H 4820 2846 50  0000 L CNN
 F 1 "R" H 4820 2755 50  0000 L CNN
 F 2 "Resistor_THT:R_Axial_DIN0207_L6.3mm_D2.5mm_P10.16mm_Horizontal" V 4680 2800 50  0001 C CNN
@@
 memWR
 $Comp
-L Device:R R38
+L Device:R R938
 U 1 1 6110429D
 P 5000 5700
-F 0 "R38" H 5070 5746 50  0000 L CNN
+F 0 "R938" H 5070 5746 50  0000 L CNN
 F 1 "R" H 5070 5655 50  0000 L CNN
 F 2 "Resistor_THT:R_Axial_DIN0207_L6.3mm_D2.5mm_P10.16mm_Horizontal" V 4930 5700 50  0001 C CNN

Commit message: route A8-A15 to U131
Parts:
- R32, R33, R34, R35, R36, R39, R40, R41, R42, R43: footprint Resistor_THT:R_Axial_DIN0207_L6.3mm_D2.5mm_P10.16mm_Horizontal -> Resistor_THT:R_Axial_DIN0204_L3.6mm_D1.6mm_P5.08mm_Horizontal
Changed lines of the file:
@@
 F 0 "R32" H 1670 4046 50  0000 L CNN
 F 1 "R" H 1670 3955 50  0000 L CNN
-F 2 "Resistor_THT:R_Axial_DIN0207_L6.3mm_D2.5mm_P10.16mm_Horizontal" V 1530 4000 50  0001 C CNN
+F 2 "Resistor_THT:R_Axial_DIN0204_L3.6mm_D1.6mm_P5.08mm_Horizontal" V 1530 4000 50  0001 C CNN
 F 3 "~" H 1600 4000 50  0001 C CNN
 	1    1600 4000
@@
 F 0 "R34" H 3420 4646 50  0000 L CNN
 F 1 "R" H 3420 4555 50  0000 L CNN
-F 2 "Resistor_THT:R_Axial_DIN0207_L6.3mm_D2.5mm_P10.16mm_Horizontal" V 3280 4600 50  0001 C CNN
+F 2 "Resistor_THT:R_Axial_DIN0204_L3.6mm_D1.6mm_P5.08mm_Horizontal" V 3280 4600 50  0001 C CNN
 F 3 "~" H 3350 4600 50  0001 C CNN
 	1    3350 4600
@@
 F 0 "R41" H 7020 3946 50  0000 L CNN
 F 1 "R" H 7020 3855 50  0000 L CNN
-F 2 "Resistor_THT:R_Axial_DIN0207_L6.3mm_D2.5mm_P10.16mm_Horizontal" V 6880 3900 50  0001 C CNN
+F 2 "Resistor_THT:R_Axial_DIN0204_L3.6mm_D1.6mm_P5.08mm_Horizontal" V 6880 3900 50  0001 C CNN
 F 3 "~" H 6950 3900 50  0001 C CNN
 	1    6950 3900
@@
 F 0 "R40" H 7020 2646 50  0000 L CNN
 F 1 "R" H 7020 2555 50  0000 L CNN
-F 2 "Resistor_THT:R_Axial_DIN0207_L6.3mm_D2.5mm_P10.16mm_Horizontal" V 6880 2600 50  0001 C CNN
+F 2 "Resistor_THT:R_Axial_DIN0204_L3.6mm_D1.6mm_P5.08mm_Horizontal" V 6880 2600 50  0001 C CNN
 F 3 "~" H 6950 2600 50  0001 C CNN
 	1    6950 2600
@@
 F 0 "R36" H 4820 1996 50  0000 L CNN
 F 1 "R" H 4820 1905 50  0000 L CNN
-F 2 "Resistor_THT:R_Axial_DIN0207_L6.3mm_D2.5mm_P10.16mm_Horizontal" V 4680 1950 50  0001 C CNN
+F 2 "Resistor_THT:R_Axial_DIN0204_L3.6mm_D1.6mm_P5.08mm_Horizontal" V 4680 1950 50  0001 C CNN
 F 3 "~" H 4750 1950 50  0001 C CNN
 	1    4750 1950
@@
 F 0 "R39" H 7020 1796 50  0000 L CNN
 F 1 "R" H 7020 1705 50  0000 L CNN
-F 2 "Resistor_THT:R_Axial_DIN0207_L6.3mm_D2.5mm_P10.16mm_Horizontal" V 6880 1750 50  0001 C CNN
+F 2 "Resistor_THT:R_Axial_DIN0204_L3.6mm_D1.6mm_P5.08mm_Horizontal" V 6880 1750 50  0001 C CNN
 F 3 "~" H 6950 1750 50  0001 C CNN
 	1    6950 1750
@@
 F 0 "R35" H 4820 1146 50  0000 L CNN
 F 1 "R" H 4820 1055 50  0000 L CNN
-F 2 "Resistor_THT:R_Axial_DIN0207_L6.3mm_D2.5mm_P10.16mm_Horizontal" V 4680 1100 50  0001 C CNN
+F 2 "Resistor_THT:R_Axial_DIN0204_L3.6mm_D1.6mm_P5.08mm_Horizontal" V 4680 1100 50  0001 C CNN
 F 3 "~" H 4750 1100 50  0001 C CNN
 	1    4750 1100
@@
 F 0 "R33" H 2620 5196 50  0000 L CNN
 F 1 "R" H 2620 5105 50  0000 L CNN
-F 2 "Resistor_THT:R_Axial_DIN0207_L6.3mm_D2.5mm_P10.16mm_Horizontal" V 2480 5150 50  0001 C CNN
+F 2 "Resistor_THT:R_Axial_DIN0204_L3.6mm_D1.6mm_P5.08mm_Horizontal" V 2480 5150 50  0001 C CNN
 F 3 "~" H 2550 5150 50  0001 C CNN
 	1    2550 5150
@@
 F 0 "R42" H 7020 5546 50  0000 L CNN
 F 1 "R" H 7020 5455 50  0000 L CNN
-F 2 "Resistor_THT:R_Axial_DIN0207_L6.3mm_D2.5mm_P10.16mm_Horizontal" V 6880 5500 50  0001 C CNN
+F 2 "Resistor_THT:R_Axial_DIN0204_L3.6mm_D1.6mm_P5.08mm_Horizontal" V 6880 5500 50  0001 C CNN
 F 3 "~" H 6950 5500 50  0001 C CNN
 	1    6950 5500
@@
 F 0 "R43" H 7020 6996 50  0000 L CNN
 F 1 "R" H 7020 6905 50  0000 L CNN
-F 2 "Resistor_THT:R_Axial_DIN0207_L6.3mm_D2.5mm_P10.16mm_Horizontal" V 6880 6950 50  0001 C CNN
+F 2 "Resistor_THT:R_Axial_DIN0204_L3.6mm_D1.6mm_P5.08mm_Horizontal" V 6880 6950 50  0001 C CNN
 F 3 "~" H 6950 6950 50  0001 C CNN
 	1    6950 6950
