File: reg_WK.sch (KiCad schematic (older format))
At the start: 35 parts, among them U179 74HC244, U180 74HC244, U192 74HC244, U193 74HC244, U213 74HC373, U214 74HC373

Commit message: more updates to HL
Connections:
- net at L197.1 (K): now also B29.9 (R8); no longer B29.2 (R1)
- net at L196.1 (K): now also B29.8 (R7); no longer B29.3 (R2)
- net at L195.1 (K): now also B29.7 (R6); no longer B29.4 (R3)
- net at L194.1 (K): now also B29.6 (R5); no longer B29.5 (R4)
- net at L193.1 (K): now also B29.5 (R4); no longer B29.6 (R5)
- net at L192.1 (K): now also B29.4 (R3); no longer B29.7 (R6)
- net at L191.1 (K): now also B29.3 (R2); no longer B29.8 (R7)
- net at L190.1 (K): now also B29.2 (R1); no longer B29.9 (R8)
Changed lines of the file:
@@
 L Device:R_Network08 RN?
 U 1 1 5E39B58B
-P 4700 4500
+P 4600 4500
 AR Path="/5CAD6F89/5E39B58B" Ref="RN?"  Part="1"
 AR Path="/5D8315BB/5E39B58B" Ref="RN?"  Part="1"
 AR Path="/5E031B2C/5E39B58B" Ref="RN?"  Part="1"
 AR Path="/5E045D26/5E39B58B" Ref="B29"  Part="1"
-F 0 "B29" H 4220 4454 50  0000 R CNN
-F 1 "2.2K" H 4220 4545 50  0000 R CNN
-F 2 "Resistor_THT:R_Array_SIP9" V 5175 4500 50  0001 C CNN
-F 3 "http://www.vishay.com/docs/31509/csc.pdf" H 4700 4500 50  0001 C CNN
-	1    4700 4500
-	1    0    0    1
+F 0 "B29" H 4120 4454 50  0000 R CNN
+F 1 "2.2K" H 4120 4545 50  0000 R CNN
+F 2 "Resistor_THT:R_Array_SIP9" V 5075 4500 50  0001 C CNN
+F 3 "http://www.vishay.com/docs/31509/csc.pdf" H 4600 4500 50  0001 C CNN
+	1    4600 4500
+	-1   0    0    1
 $EndComp
 Wire Wire Line
@@
 L power:GND #PWR?
 U 1 1 5E39B5B5
-P 4300 4700
+P 5000 4700
 AR Path="/5CAD6F89/5E39B5B5" Ref="#PWR?"  Part="1"
 AR Path="/5D8315BB/5E39B5B5" Ref="#PWR?"  Part="1"
 AR Path="/5E031B2C/5E39B5B5" Ref="#PWR?"  Part="1"
 AR Path="/5E045D26/5E39B5B5" Ref="#PWR0121"  Part="1"
-F 0 "#PWR0121" H 4300 4450 50  0001 C CNN
-F 1 "GND" H 4305 4527 50  0000 C CNN
-F 2 "" H 4300 4700 50  0001 C CNN
-F 3 "" H 4300 4700 50  0001 C CNN
-	1    4300 4700
+F 0 "#PWR0121" H 5000 4450 50  0001 C CNN
+F 1 "GND" H 5005 4527 50  0000 C CNN
+F 2 "" H 5000 4700 50  0001 C CNN
+F 3 "" H 5000 4700 50  0001 C CNN
+	1    5000 4700
 	1    0    0    -1
 $EndComp
